File: microjuice/microjuice.kicad_sch (KiCad schematic)
At the start: 27 parts, among them J1 USB_A, J2 USB_B_Micro, J3 Conn_01x03_Male, J4 Conn_01x03_Male, J5 Conn_01x03_Male, U1 AMS1117-3.3

Commit message: Add v2
Parts:
- removed C1: 10u, Capacitor_Tantalum_SMD:CP_EIA-3216-18_Kemet-A, symbol Device:C
- removed C2: (no value), symbol Device:C
- removed J2: USB_B_Micro, Connector_USB:USB_Micro-B_Molex-105017-0001, symbol Connector:USB_B_Micro
- added C1: 100u, Capacitor_SMD:CP_Elec_6.3x5.4_Nichicon, symbol Device:C_Polarized
- added C2, C6: 10u, Capacitor_Tantalum_SMD:CP_EIA-3216-18_Kemet-A, symbol Device:C_Polarized
- added C3, C4, C5: 470n, Capacitor_SMD:C_0603_1608Metric, symbol Device:C
- added H12, H13, H14, H15: MountingHole, MountingHole:MountingHole_3.2mm_M3, symbol Mechanical:MountingHole
- added JP1, JP2, JP3: SolderJumper_2_Open, Jumper:SolderJumper-2_P1.3mm_Open_TrianglePad1.0x1.5mm, symbol Jumper:SolderJumper_2_Open
- added U2, U3, U4: 74AHCT1G125, Package_TO_SOT_SMD:SOT-23-5, symbol 74xGxx:74AHCT1G125
- H1, H10, H11, H2, H3, H6: footprint MountingHole:MountingHole_3.7mm_Pad -> footprints:SpuntDira; now left out of the parts list
- H4, H5, H7, H8, H9: footprint MountingHole:MountingHole_3.7mm_Pad -> footprints:SMTSO30; LCSC (none) -> C2916371
- J1: now left out of the parts list
Connections:
- net GND: now also J3.1 (Pin_1), J4.1 (Pin_1), J5.1 (Pin_1), C1.2, C2.2, C3.1, C4.1, C5.1, C6.2, U2.1, U2.3 (GND), U3.1, U3.3 (GND), U4.1, U4.3 (GND); no longer J1.5 (Shield), J3.3 (Pin_3), J4.3 (Pin_3), J5.3 (Pin_3)
- net VBUS: now also C1.1, C2.1, C3.2, C4.2, C5.2, U2.5 (VCC), U3.5 (VCC), U4.5 (VCC)
- net at D2.1, H1.1, R1.2: now also JP1.2 (B), U2.2; no longer J3.1 (Pin_1)
- net at D2.2, H2.1, R2.2: now also JP2.2 (B), U3.2; no longer J4.1 (Pin_1)
- net at D1.2 (A), U1.2 (VO): now also C6.1
- net at D3.2, H3.1, R3.2: now also JP3.2 (B), U4.2; no longer J5.1 (Pin_1)
- new net: J5.3 (Pin_3), JP3.1 (A), U4.4
- new net: J4.3 (Pin_3), JP2.1 (A), U3.4
- new net: J3.3 (Pin_3), JP1.1 (A), U2.4
- no-connect marks 0 -> 1
Other:
- moved on the sheet: D1, D2, D3, D4, H1, H10, H11, H2, H3, H4, H5, H6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
